File: 2bitAdder.sch (KiCad schematic (older format))
At the start: 18 parts, among them J1 Conn_01x02_Male, SW1 SW_Push, SW2 SW_Push, SW3 SW_Push, SW4 SW_Push, U1 74LS386, U2 74LS08, U3 74LS32

Commit message: Update netlist
Parts:
- R1, R4, R5: value R -> 220
- R2, R3, R6, R7: value R -> 10K
Changed lines of the file:
@@
 LIBS:contrib
 LIBS:valves
+LIBS:2bitAdder-cache
 EELAYER 25 0
 EELAYER END
@@
 P 9100 1200
 F 0 "R2" V 9180 1200 50  0000 C CNN
-F 1 "R" V 9100 1200 50  0000 C CNN
+F 1 "10K" V 9100 1200 50  0000 C CNN
 F 2 "Resistors_THT:R_Axial_DIN0207_L6.3mm_D2.5mm_P10.16mm_Horizontal" V 9030 1200 50  0001 C CNN
 F 3 "" H 9100 1200 50  0001 C CNN
@@
 P 10700 1200
 F 0 "R6" V 10780 1200 50  0000 C CNN
-F 1 "R" V 10700 1200 50  0000 C CNN
+F 1 "10K" V 10700 1200 50  0000 C CNN
 F 2 "Resistors_THT:R_Axial_DIN0207_L6.3mm_D2.5mm_P10.16mm_Horizontal" V 10630 1200 50  0001 C CNN
 F 3 "" H 10700 1200 50  0001 C CNN
@@
 P 9100 1900
 F 0 "R3" V 9180 1900 50  0000 C CNN
-F 1 "R" V 9100 1900 50  0000 C CNN
+F 1 "10K" V 9100 1900 50  0000 C CNN
 F 2 "Resistors_THT:R_Axial_DIN0207_L6.3mm_D2.5mm_P10.16mm_Horizontal" V 9030 1900 50  0001 C CNN
 F 3 "" H 9100 1900 50  0001 C CNN
@@
 P 10700 1900
 F 0 "R7" V 10780 1900 50  0000 C CNN
-F 1 "R" V 10700 1900 50  0000 C CNN
+F 1 "10K" V 10700 1900 50  0000 C CNN
 F 2 "Resistors_THT:R_Axial_DIN0207_L6.3mm_D2.5mm_P10.16mm_Horizontal" V 10630 1900 50  0001 C CNN
 F 3 "" H 10700 1900 50  0001 C CNN
@@
 P 8850 3150
 F 0 "R1" V 8930 3150 50  0000 C CNN
-F 1 "R" V 8850 3150 50  0000 C CNN
+F 1 "220" V 8850 3150 50  0000 C CNN
 F 2 "Resistors_THT:R_Axial_DIN0207_L6.3mm_D2.5mm_P10.16mm_Horizontal" V 8780 3150 50  0001 C CNN
 F 3 "" H 8850 3150 50  0001 C CNN
@@
 P 9400 3150
 F 0 "R4" V 9480 3150 50  0000 C CNN
-F 1 "R" V 9400 3150 50  0000 C CNN
+F 1 "220" V 9400 3150 50  0000 C CNN
 F 2 "Resistors_THT:R_Axial_DIN0207_L6.3mm_D2.5mm_P10.16mm_Horizontal" V 9330 3150 50  0001 C CNN
 F 3 "" H 9400 3150 50  0001 C CNN
@@
 P 9950 3150
 F 0 "R5" V 10030 3150 50  0000 C CNN
-F 1 "R" V 9950 3150 50  0000 C CNN
+F 1 "220" V 9950 3150 50  0000 C CNN
 F 2 "Resistors_THT:R_Axial_DIN0207_L6.3mm_D2.5mm_P10.16mm_Horizontal" V 9880 3150 50  0001 C CNN
 F 3 "" H 9950 3150 50  0001 C CNN
