File: 2bitAdder.kicad_pcb (KiCad board)
At the start: 2 copper layers, 53.3 x 71.1 mm, 24 parts, among them J1 Conn_01x02_Male, SW1 SW_Push, SW2 SW_Push, SW3 SW_Push, SW4 SW_Push, U1 74LS386, U2 74LS08, U3 74LS32

Commit message: Added +/- indicator to power pins
Other:
- board text added: "- +"
Changed lines of the file:
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@@
     (links 55)
     (no_connects 0)
-    (area 70.604761 74.412499 154.185239 148.55)
+    (area 70.604761 74.412499 154.185239 146.567502)
     (thickness 1.6)
-    (drawings 6)
+    (drawings 7)
     (tracks 240)
     (zones 0)
@@
       (outputformat 5)
       (mirror false)
-      (drillshape 0)
+      (drillshape 1)
       (scaleselection 1)
       (outputdirectory svg/))
@@
       (solder_mask_margin 0.77) (clearance 0.77))
   )
+  (gr_text "-\n+" (at 130.81 88.9) (layer F.Cu)
+    (effects (font (size 1.5 1.5) (thickness 0.3)))
+  )
   (gr_line (start 86.36 146.05) (end 86.36 74.93) (angle 90) (layer Edge.Cuts) (width 0.15))
